File: hardware/QTouchShield/QTouchShield.sch (EAGLE design)
At the start: 114 parts, among them IC1 AT32UC3C0512C, U1 ARDUINO-MEGALITE

Commit message: Changed LQFP-144 footprint.
Ripped up LQFP-144 package footprint and replaced by footprint from an
offical EagleCAD library.
Parts:
- IC1: value AT32UC3C0512C -> AT32UC3C0512CJEDEC-MS-026; device atmel-AVR32:AT32UC3C0512C -> atmel-AVR32:AT32UC3C0512CJEDEC-MS-026
Changed lines of the file:
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@@
 </classes>
 <parts>
-<part name="IC1" library="atmel-AVR32" deviceset="AT32UC3C0512C" device=""/>
+<part name="IC1" library="atmel-AVR32" deviceset="AT32UC3C0512C" device="JEDEC-MS-026"/>
 <part name="U1" library="SparkFun" deviceset="ARDUINO-MEGA" device="LITE"/>
 <part name="JP1" library="pinhead" deviceset="PINHD-1X3" device="" value="COMMS_SELECT"/>
